Commit message: EXP4: Jump Height

File: models/planar_walker_2.urdf (robot description, URDF)
Before this commit: robot KneedCompassGait, 13 links, 12 joints
Links:
- link left_lower_leg_mass: mass 0.6 -> 0.5
- link left_upper_leg_mass: mass 1.0 -> 1.5
- link right_lower_leg_mass: mass 0.3 -> 0.5
- link right_upper_leg_mass: mass 1.7 -> 1.5
- link torso_mass: mass 55 -> 51
